Commit message: fuser 코드 추가

File: install/carsa_gazebo/share/carsa_gazebo/urdf/erp42.xacro (robot description, xacro)
@@ -1,82 +1 @@
-<?xml version="1.0"?>
-<robot xmlns:xacro="http://ros.org/wiki/xacro" name="erp42_scmc">
-    <!-- Include files -->
-    <xacro:include filename="$(find erp42_gazebo)/urdf/erp42_gazebo_control.xacro"/>
-    <xacro:include filename="$(find carsa_gazebo)/urdf/xsens_mti3.xacro"/>
-    <xacro:include filename="$(find carsa_gazebo)/urdf/ublox_zed_f9p.xacro"/>
-    <xacro:include filename="$(find carsa_gazebo)/urdf/velodyne_vlp_32c.xacro"/>
-    <xacro:include filename="$(find carsa_gazebo)/urdf/logitech_c930.xacro"/>
-    <xacro:include filename="$(find carsa_gazebo)/urdf/logitech_c920.xacro"/>
-    <!-- ERP42 model description and gazebo control settings -->
-    <xacro:erp42_gazebo_control publish_odometry = "true"/>
-    <!-- Xsens IMU -->
-    <xacro:xsens_mti3
-        parent_link = "base_link"
-        sensor_name = "xsens"
-        x           = "0.0"
-        y           = "0.0"
-        z           = "0.5"
-        roll        = "0.0"
-        pitch       = "0.0"
-        yaw         = "0.0"
-    />
-    <!-- Ublox zed f9p GPS -->
-    <xacro:ublox_zed_f9p
-        parent_link = "base_link"
-        sensor_name = "ublox_gps"
-        x           = "0.0"
-        y           = "0.0"
-        z           = "1.2"
-        roll        = "0.0"
-        pitch       = "0.0"
-        yaw         = "0.0"
-    />
-    <!-- Velodyne LiDAR -->
-    <xacro:velodyne_vlp_32c
-        parent_link  = "base_link"
-        sensor_name  = "velodyne"
-        visualize    = "false"
-        x            = "0.0"
-        y            = "0.0"
-        z            = "1.0"
-        roll         = "0.0"
-        pitch        = "0.0"
-        yaw          = "0.0"
-    />
-    <!-- Logitech C920 camera : traffic_light -->
-    <xacro:logitech_c920
-        parent_link  = "base_link"
-        sensor_name  = "logitech_c920_traffic_light"
-        visualize    = "true"
-        x            = "0.25"
-        y            = "0.0"
-        z            = "0.75"
-        roll         = "0.0"
-        pitch        = "-20.0"
-        yaw          = "0.0"
-    />
-    <!-- Logitech C930 camera : left side -->
-    <xacro:logitech_c930
-        parent_link  = "base_link"
-        sensor_name  = "logitech_c930_left"
-        visualize    = "true"
-        x            = "0.0"
-        y            = "0.40"
-        z            = "0.75"
-        roll         = "0.0"
-        pitch        = "0.0"
-        yaw          = "30.0"
-    />
-    <!-- Logitech C930 camera : right side -->
-    <xacro:logitech_c930
-        parent_link  = "base_link"
-        sensor_name  = "logitech_c930_right"
-        visualize    = "true"
-        x            = "0.0"
-        y            = "-0.40"
-        z            = "0.75"
-        roll         = "0.0"
-        pitch        = "0.0"
-        yaw          = "-30.0"
-    />
-</robot>
+/home/kimsohee/ev-1-5/ev-Autonomous-Vehicle-1-5/carsa_gazebo/urdf/erp42.xacro

File: install/carsa_gazebo/share/carsa_gazebo/urdf/logitech_c920.xacro (robot description, xacro)
@@ -1,86 +1 @@
-<?xml version="1.0" ?>
-<robot xmlns:xacro="http://ros.org/wiki/xacro">
-    <!-- Logitech C920 camera -->
-    <xacro:macro name="logitech_c920" params="parent_link sensor_name visualize x y z roll pitch yaw">
-        <!-- Variables -->
-        <xacro:property name="frame_length" value="0.025"/>
-        <xacro:property name="frame_width"  value="0.090"/>
-        <xacro:property name="frame_height" value="0.028"/>
-        <!-- Links -->
-        <link name="${sensor_name}">
-            <!-- Mesh -->
-            <visual>
-                <origin xyz="0 0 ${frame_height/2}" rpy="0 0 0" />
-                <geometry>
-                    <mesh filename="file://$(find carsa_gazebo)/meshes/logitech_c920.dae" scale="0.001 0.001 0.001"/>
-                </geometry>
-            </visual>
-        </link>
-        <link name="${sensor_name}_optical">
-            <!-- Mesh -->
-            <visual>
-                <origin xyz="0 0 0" rpy="0 0 0" />
-                <geometry>
-                    <mesh filename="file://$(find carsa_gazebo)/meshes/logitech_camera_lens.dae" scale="0.001 0.001 0.001"/>
-                </geometry>
-            </visual>
-        </link>
-        <!-- Joints -->
-        <joint name="${sensor_name}_joint" type="fixed">
-            <!-- Origin -->
-            <origin xyz="${x} ${y} ${z}" rpy="${radians(roll)} ${radians(pitch)} ${radians(yaw)}" />
-            <!-- Frame ID -->
-            <parent link="${parent_link}" />
-            <child link="${sensor_name}" />
-        </joint>
-        <joint name="${sensor_name}_optical_joint" type="fixed">
-            <!-- Origin -->
-            <!-- <origin xyz="0 0 ${frame_height/2}" rpy="${-pi/2} 0 ${-pi/2}" /> -->
-            <origin xyz="0 0 ${frame_height/2}" rpy="0 0 0" />
-            <!-- Frame ID -->
-            <parent link="${sensor_name}" />
-            <child link="${sensor_name}_optical" />
-        </joint>
-        <!-- Gazebo plugin -->
-        <gazebo reference="${sensor_name}_optical">
-            <!-- Sensor properties -->
-            <sensor name="${sensor_name}" type="camera">
-                <!-- Topic -->
-                <update_rate>30</update_rate>
-                <always_on>true</always_on>
-                <visualize>${visualize}</visualize>
-                <!-- Optical -->
-                <camera>
-                    <!-- FOV-->
-                    <horizontal_fov>0.911384</horizontal_fov>
-                    <!-- Data formats -->
-                    <image>
-                        <width>640</width>
-                        <height>480</height>
-                        <format>R8G8B8</format>
-                    </image>
-                    <!-- Detection area -->
-                    <clip>
-                        <near>0.05</near>
-                        <far>100.0</far>
-                    </clip>
-                    <!-- Distortion -->
-                    <!--
-                    <distortion>
-                        <k1>0.162875</k1><k2>-0.287212</k2><k3>0.0</k3>
-                        <p1>0.000692</p1><p2>-0.000678</p2>
-                        <center><x>291.5055</x><y>222.6638</y></center>
-                    </distortion>
-                    -->
-                </camera>
-                <!-- Gazebo ROS camera plugin -->
-                <plugin name="${sensor_name}_plugin" filename="libgazebo_ros_camera.so">
-                    <camera_name>${sensor_name}</camera_name>
-                    <image_topic_name>${sensor_name}/image_raw</image_topic_name>
-                    <camera_info_topic_name>${sensor_name}/camera_info</camera_info_topic_name>
-                    <frame_name>${sensor_name}_optical</frame_name>
-                </plugin>
-            </sensor>
-        </gazebo>
-    </xacro:macro>
-</robot>
+/home/kimsohee/ev-1-5/ev-Autonomous-Vehicle-1-5/carsa_gazebo/urdf/logitech_c920.xacro

File: install/carsa_gazebo/share/carsa_gazebo/urdf/logitech_c930.xacro (robot description, xacro)
@@ -1,86 +1 @@
-<?xml version="1.0" ?>
-<robot xmlns:xacro="http://ros.org/wiki/xacro">
-    <!-- Logitech C930 camera -->
-    <xacro:macro name="logitech_c930" params="parent_link sensor_name visualize x y z roll pitch yaw">
-        <!-- Variables -->
-        <xacro:property name="frame_length" value="0.025"/>
-        <xacro:property name="frame_width"  value="0.090"/>
-        <xacro:property name="frame_height" value="0.028"/>
-        <!-- Links -->
-        <link name="${sensor_name}">
-            <!-- Mesh -->
-            <visual>
-                <origin xyz="0 0 ${frame_height/2}" rpy="0 0 0" />
-                <geometry>
-                    <mesh filename="file://$(find carsa_gazebo)/meshes/logitech_c930.dae" scale="0.001 0.001 0.001"/>
-                </geometry>
-            </visual>
-        </link>
-        <link name="${sensor_name}_optical">
-            <!-- Mesh -->
-            <visual>
-                <origin xyz="0 0 0" rpy="0 0 0" />
-                <geometry>
-                    <mesh filename="file://$(find carsa_gazebo)/meshes/logitech_camera_lens.dae" scale="0.001 0.001 0.001"/>
-                </geometry>
-            </visual>
-        </link>
-        <!-- Joints -->
-        <joint name="${sensor_name}_joint" type="fixed">
-            <!-- Origin -->
-            <origin xyz="${x} ${y} ${z}" rpy="${radians(roll)} ${radians(pitch)} ${radians(yaw)}" />
-            <!-- Frame ID -->
-            <parent link="${parent_link}" />
-            <child link="${sensor_name}" />
-        </joint>
-        <joint name="${sensor_name}_optical_joint" type="fixed">
-            <!-- Origin -->
-            <!-- <origin xyz="0 0 ${frame_height/2}" rpy="${-pi/2} 0 ${-pi/2}" /> -->
-            <origin xyz="0 0 ${frame_height/2}" rpy="0 0 0" />
-            <!-- Frame ID -->
-            <parent link="${sensor_name}" />
-            <child link="${sensor_name}_optical" />
-        </joint>
-        <!-- Gazebo plugin -->
-        <gazebo reference="${sensor_name}_optical">
-            <!-- Sensor properties -->
-            <sensor name="${sensor_name}" type="camera">
-                <!-- Topic -->
-                <update_rate>30</update_rate>
-                <always_on>true</always_on>
-                <visualize>${visualize}</visualize>
-                <!-- Optical -->
-                <camera>
-                    <!-- FOV-->
-                    <horizontal_fov>1.167485</horizontal_fov>
-                    <!-- Data formats -->
-                    <image>
-                        <width>640</width>
-                        <height>480</height>
-                        <format>R8G8B8</format>
-                    </image>
-                    <!-- Detection area -->
-                    <clip>
-                        <near>0.05</near>
-                        <far>100.0</far>
-                    </clip>
-                    <!-- Distortion -->
-                    <!--
-                    <distortion>
-                        <k1>0.162875</k1><k2>-0.287212</k2><k3>0.0</k3>
-                        <p1>0.000692</p1><p2>-0.000678</p2>
-                        <center><x>291.5055</x><y>222.6638</y></center>
-                    </distortion>
-                    -->
-                </camera>
-                <!-- Gazebo ROS camera plugin -->
-                <plugin name="${sensor_name}_plugin" filename="libgazebo_ros_camera.so">
-                    <camera_name>${sensor_name}</camera_name>
-                    <image_topic_name>${sensor_name}/image_raw</image_topic_name>
-                    <camera_info_topic_name>${sensor_name}/camera_info</camera_info_topic_name>
-                    <frame_name>${sensor_name}_optical</frame_name>
-                </plugin>
-            </sensor>
-        </gazebo>
-    </xacro:macro>
-</robot>
+/home/kimsohee/ev-1-5/ev-Autonomous-Vehicle-1-5/carsa_gazebo/urdf/logitech_c930.xacro

File: install/carsa_gazebo/share/carsa_gazebo/urdf/t870.xacro (robot description, xacro)
@@ -1,88 +1 @@
-<?xml version="1.0"?>
-<robot xmlns:xacro="http://ros.org/wiki/xacro" name="erp42_scmc">
-    <!-- Include files -->
-    <xacro:include filename="$(find erp42_gazebo)/urdf/erp42_gazebo_control.xacro"/>
-    <!-- <xacro:include filename="$(find carsa_gazebo)/urdf/xsens_mti3.xacro"/> -->
-    <!-- <xacro:include filename="$(find carsa_gazebo)/urdf/ublox_zed_f9p.xacro"/> -->
-    <xacro:include filename="$(find carsa_gazebo)/urdf/velodyne_vlp_32c.xacro"/>
-    <!-- <xacro:include filename="$(find carsa_gazebo)/urdf/logitech_c930.xacro"/> -->
-    <!-- ERP42 model description and gazebo control settings -->
-    <xacro:erp42_gazebo_control publish_odometry = "true"/>
-    <!-- Xsens IMU -->
-    <!-- <xacro:xsens_mti3
-        parent_link = "base_link"
-        sensor_name = "xsens"
-        x           = "0.0"
-        y           = "0.0"
-        z           = "0.5"
-        roll        = "0.0"
-        pitch       = "0.0"
-        yaw         = "0.0"
-    /> -->
-    <!-- Ublox zed f9p GPS -->
-    <!-- <xacro:ublox_zed_f9p
-        parent_link = "base_link"
-        sensor_name = "ublox_gps"
-        x           = "0.0"
-        y           = "0.0"
-        z           = "1.2"
-        roll        = "0.0"
-        pitch       = "0.0"
-        yaw         = "0.0"
-    /> -->
-    <!-- Velodyne LiDAR -->
-    <!-- <xacro:velodyne_vlp_16c
-        parent_link  = "base_link"
-        sensor_name  = "velodyne"
-        visualize    = "false"
-        x            = "0.0"
-        y            = "0.0"
-        z            = "0.90"
-        roll         = "0.0"
-        pitch        = "0.0"
-        yaw          = "0.0"
-    /> -->
-    <xacro:velodyne_vlp_32c
-        parent_link="base_link"
-        sensor_name="velodyne"
-        visualize="false"
-        x="0.0" y="0.0" z="0.90"
-        roll="0.0" pitch="0.0" yaw="0.0"
-    />
-    <!-- Logitech C920 camera : traffic_light -->
-    <!-- <xacro:logitech_c920
-        parent_link  = "base_link"
-        sensor_name  = "logitech_c920_traffic_light"
-        visualize    = "true"
-        x            = "0.25"
-        y            = "0.0"
-        z            = "0.75"
-        roll         = "0.0"
-        pitch        = "-20.0"
-        yaw          = "0.0"
-    /> -->
-    <!-- Logitech C930 camera : left side -->
-    <!-- <xacro:logitech_c930
-        parent_link  = "base_link"
-        sensor_name  = "logitech_c930_left"
-        visualize    = "true"
-        x            = "0.0"
-        y            = "0.40"
-        z            = "0.75"
-        roll         = "0.0"
-        pitch        = "0.0"
-        yaw          = "30.0"
-    /> -->
-    <!-- Logitech C930 camera : right side -->
-    <!-- <xacro:logitech_c930
-        parent_link  = "base_link"
-        sensor_name  = "logitech_c930_right"
-        visualize    = "true"
-        x            = "0.0"
-        y            = "-0.40"
-        z            = "0.75"
-        roll         = "0.0"
-        pitch        = "0.0"
-        yaw          = "-30.0"
-    /> -->
-</robot>
+/home/kimsohee/ev-1-5/ev-Autonomous-Vehicle-1-5/carsa_gazebo/urdf/t870.xacro

File: install/carsa_gazebo/share/carsa_gazebo/urdf/ublox_zed_f9p.xacro (robot description, xacro)
@@ -1,78 +1 @@
-<?xml version="1.0" ?>
-<robot xmlns:xacro="http://ros.org/wiki/xacro">
-    <!-- Ublox zed f9p GPS -->
-    <xacro:macro name="ublox_zed_f9p" params="parent_link sensor_name x y z roll pitch yaw">
-        <!-- Link -->
-        <link name="${sensor_name}">
-            <!-- Mesh -->
-            <visual>
-                <origin xyz="0 0 0" rpy="0 0 0" />
-                <geometry>
-                    <mesh filename="file://$(find carsa_gazebo)/meshes/gps_antenna.dae" scale="0.001 0.001 0.001"/>
-                </geometry>
-            </visual>
-        </link>
-        <!-- Joint -->
-        <joint name="${sensor_name}_joint" type="fixed">
-            <!-- Origin -->
-            <origin xyz="${x} ${y} ${z}" rpy="${radians(roll)} ${radians(pitch)} ${radians(yaw)}" />
-            <!-- Frame ID -->
-            <parent link="${parent_link}" />
-            <child link="${sensor_name}" />
-        </joint>
-        <!-- Gazebo plugin -->
-        <gazebo reference="${sensor_name}">
-            <!-- Sensor properties -->
-            <sensor name="${sensor_name}" type="gps">
-                <always_on>true</always_on>
-                <update_rate>10</update_rate>
-                <visualize>false</visualize>
-                <!-- Data formats -->
-                <gps>
-                    <!-- Position sensing -->
-                    <position_sensing>
-                        <!-- Horizontal -->
-                        <horizontal>
-                            <noise type="gaussian">
-                                <mean>0.0</mean>
-                                <stddev>0.0014</stddev>
-                            </noise>
-                        </horizontal>
-                        <!-- Vertical -->
-                        <vertical>
-                            <noise type="gaussian">
-                                <mean>0.0</mean>
-                                <stddev>0.0014</stddev>
-                            </noise>
-                        </vertical>
-                    </position_sensing>
-                    <!-- Velocity sensing -->
-                    <velocity_sensing>
-                        <!-- Horizontal -->
-                        <horizontal>
-                            <noise type="gaussian">
-                                <mean>0.0</mean>
-                                <stddev>0.0014</stddev>
-                            </noise>
-                        </horizontal>
-                        <!-- Vertical -->
-                        <vertical>
-                            <noise type="gaussian">
-                                <mean>0.0</mean>
-                                <stddev>0.0014</stddev>
-                            </noise>
-                        </vertical>
-                    </velocity_sensing>
-                </gps>
-                <!-- Gazebo ROS plugin -->
-                <plugin name="${sensor_name}_plugin" filename="libgazebo_ros_gps_sensor.so">
-                    <ros>
-                        <remapping>~/out:=${sensor_name}/fix</remapping>
-                        <remapping>~/vel:=${sensor_name}/velocity</remapping>
-                    </ros>
-                    <frame_name>${sensor_name}</frame_name>
-                </plugin>
-            </sensor>
-        </gazebo>
-    </xacro:macro>
-</robot>
+/home/kimsohee/ev-1-5/ev-Autonomous-Vehicle-1-5/carsa_gazebo/urdf/ublox_zed_f9p.xacro
