Commit message: fuser 코드 추가

File: install/carsa_gazebo/share/carsa_gazebo/urdf/velodyne_vlp_16c.xacro (robot description, xacro)
@@ -1,119 +1 @@
-<?xml version="1.0" ?>
-<robot xmlns:xacro="http://ros.org/wiki/xacro">
-    <!-- Velodyne VLP32C LiDAR -->
-    <xacro:macro name="velodyne_vlp_16c" params="parent_link sensor_name visualize x y z roll pitch yaw">
-        <!-- Variables -->
-        <xacro:property name = "lens_radius"  value = "0.050" />
-        <xacro:property name = "lens_length"  value = "0.055" />
-        <xacro:property name = "frame_radius" value = "0.052" />
-        <xacro:property name = "frame_length" value = "0.015" />
-        <!-- Links -->
-        <link name="${sensor_name}">
-            <!-- Mesh -->
-            <visual>
-                <origin xyz="0 0 ${frame_length/2}" rpy="0 0 0" />
-                <geometry>
-                    <cylinder radius = "${frame_radius}" length = "${frame_length}"/>
-                </geometry>
-                <material name="silver">
-                    <color rgba="0.85 0.85 0.85 1.0"/>
-                </material>
-            </visual>
-            <visual>
-                <origin xyz="0 0 ${3*frame_length/2 + lens_length}" rpy="0 0 0" />
-                <geometry>
-                    <cylinder radius = "${frame_radius}" length = "${frame_length}"/>
-                </geometry>
-                <material name="silver">
-                    <color rgba="0.85 0.85 0.85 1.0"/>
-                </material>
-            </visual>
-        </link>
-        <link name="${sensor_name}_optical">
-            <!-- Mesh -->
-            <visual>
-                <origin xyz="0 0 0" rpy="0 0 0" />
-                <geometry>
-                    <cylinder radius = "${lens_radius}" length = "${lens_length}"/>
-                </geometry>
-                    <material name="aquablue" >
-                        <color rgba="0.00784313725490196 0.8470588235294118 0.9137254901960784 1.0" />
-                    </material>
-            </visual>
-        </link>
-        <!-- Joints -->
-        <joint name="${sensor_name}_joint" type="fixed">
-            <!-- Origin -->
-            <origin xyz="${x} ${y} ${z}" rpy="${radians(roll)} ${radians(pitch)} ${radians(yaw)}" />
-            <!-- Frame ID -->
-            <parent link="${parent_link}" />
-            <child link="${sensor_name}" />
-        </joint>
-        <joint name="${sensor_name}_optical_joint" type="fixed">
-            <!-- Origin -->
-            <origin xyz="0 0 ${frame_length + lens_length/2}" rpy="0 0 0" />
-            <!-- Frame ID -->
-            <parent link="${sensor_name}" />
-            <child link="${sensor_name}_optical" />
-        </joint>
-        <!-- Gazebo plugin -->
-        <gazebo reference="${sensor_name}">
-            <!-- Mesh -->
-            <material>Gazebo/Gray</material>
-        </gazebo>
-        <!-- Gazebo plugin -->
-        <gazebo reference="${sensor_name}_optical">
-            <!-- Mesh -->
-            <material>Gazebo/Blue</material>
-            <!-- Sensor properties -->
-            <sensor name="${sensor_name}" type="gpu_ray">
-                <!-- Options -->
-                <update_rate>10</update_rate>
-                <always_on>true</always_on>
-	            <visualize>${visualize}</visualize>
-                <!-- Data formats -->
-                <ray>
-                    <scan>
-                        <!-- Horizontal detection area -->
-                        <horizontal>
-                            <samples>1800</samples>
-                            <resolution>1</resolution>
-                            <min_angle>-3.141592653589793</min_angle>
-                            <max_angle> 3.141592653589793</max_angle>
-                        </horizontal>
-                        <!-- Vertical detection area -->
-                        <vertical>
-                            <samples>16</samples>
-                            <resolution>1</resolution>
-                            <min_angle>-0.2617993877991494</min_angle>
-                            <max_angle> 0.2617993877991494</max_angle>
-                        </vertical>
-                    </scan>
-                    <!-- Range area -->
-                    <range>
-                        <min>1.0</min>
-                        <max>50.0</max>
-                        <resolution>0.002</resolution>
-                    </range>
-                    <!-- Noise -->
-                    <noise>
-                        <type>gaussian</type>
-                        <mean>0.0</mean>
-                        <stddev>0.0025</stddev>
-                    </noise>
-                </ray>
-                <!-- Gazebo ROS plugin -->
-                <plugin name="${sensor_name}_plugin" filename="libgazebo_ros_velodyne_laser.so">
-                    <ros>
-                        <remapping>~/out:=/${sensor_name}_points</remapping>
-                    </ros>
-                    <output_type>sensor_msgs/PointCloud2</output_type>
-                    <frame_name>${sensor_name}_optical</frame_name>
-                    <organize_cloud>false</organize_cloud>
-                    <min_range>1.0</min_range>
-                    <max_range>50.0</max_range>
-                </plugin>
-            </sensor>
-        </gazebo>
-    </xacro:macro>
-</robot>
+/home/kimsohee/ev-1-5/ev-Autonomous-Vehicle-1-5/carsa_gazebo/urdf/velodyne_vlp_16c.xacro

File: install/carsa_gazebo/share/carsa_gazebo/urdf/velodyne_vlp_32c.xacro (robot description, xacro)
@@ -1,119 +1 @@
-<?xml version="1.0" ?>
-<robot xmlns:xacro="http://ros.org/wiki/xacro">
-    <!-- Velodyne VLP32C LiDAR -->
-    <xacro:macro name="velodyne_vlp_32c" params="parent_link sensor_name visualize x y z roll pitch yaw">
-        <!-- Variables -->
-        <xacro:property name = "lens_radius"  value = "0.050" />
-        <xacro:property name = "lens_length"  value = "0.055" />
-        <xacro:property name = "frame_radius" value = "0.052" />
-        <xacro:property name = "frame_length" value = "0.015" />
-        <!-- Links -->
-        <link name="${sensor_name}">
-            <!-- Mesh -->
-            <visual>
-                <origin xyz="0 0 ${frame_length/2}" rpy="0 0 0" />
-                <geometry>
-                    <cylinder radius = "${frame_radius}" length = "${frame_length}"/>
-                </geometry>
-                <material name="silver">
-                    <color rgba="0.85 0.85 0.85 1.0"/>
-                </material>
-            </visual>
-            <visual>
-                <origin xyz="0 0 ${3*frame_length/2 + lens_length}" rpy="0 0 0" />
-                <geometry>
-                    <cylinder radius = "${frame_radius}" length = "${frame_length}"/>
-                </geometry>
-                <material name="silver">
-                    <color rgba="0.85 0.85 0.85 1.0"/>
-                </material>
-            </visual>
-        </link>
-        <link name="${sensor_name}_optical">
-            <!-- Mesh -->
-            <visual>
-                <origin xyz="0 0 0" rpy="0 0 0" />
-                <geometry>
-                    <cylinder radius = "${lens_radius}" length = "${lens_length}"/>
-                </geometry>
-                    <material name="aquablue" >
-                        <color rgba="0.00784313725490196 0.8470588235294118 0.9137254901960784 1.0" />
-                    </material>
-            </visual>
-        </link>
-        <!-- Joints -->
-        <joint name="${sensor_name}_joint" type="fixed">
-            <!-- Origin -->
-            <origin xyz="${x} ${y} ${z}" rpy="${radians(roll)} ${radians(pitch)} ${radians(yaw)}" />
-            <!-- Frame ID -->
-            <parent link="${parent_link}" />
-            <child link="${sensor_name}" />
-        </joint>
-        <joint name="${sensor_name}_optical_joint" type="fixed">
-            <!-- Origin -->
-            <origin xyz="0 0 ${frame_length + lens_length/2}" rpy="0 0 0" />
-            <!-- Frame ID -->
-            <parent link="${sensor_name}" />
-            <child link="${sensor_name}_optical" />
-        </joint>
-        <!-- Gazebo plugin -->
-        <gazebo reference="${sensor_name}">
-            <!-- Mesh -->
-            <material>Gazebo/Gray</material>
-        </gazebo>
-        <!-- Gazebo plugin -->
-        <gazebo reference="${sensor_name}_optical">
-            <!-- Mesh -->
-            <material>Gazebo/Blue</material>
-            <!-- Sensor properties -->
-            <sensor name="${sensor_name}" type="gpu_ray">
-                <!-- Options -->
-                <update_rate>20</update_rate>
-                <always_on>true</always_on>
-	            <visualize>${visualize}</visualize>
-                <!-- Data formats -->
-                <ray>
-                    <scan>
-                        <!-- Horizontal detection area -->
-                        <horizontal>
-                            <samples>2250</samples>
-                            <resolution>1</resolution>
-                            <min_angle>-3.141592653589793</min_angle>
-                            <max_angle> 3.141592653589793</max_angle>
-                        </horizontal>
-                        <!-- Vertical detection area -->
-                        <vertical>
-                            <samples>32</samples>
-                            <resolution>1</resolution>
-                            <min_angle>-0.4363323129985824</min_angle>
-                            <max_angle> 0.2617993877991494</max_angle>
-                        </vertical>
-                    </scan>
-                    <!-- Range area -->
-                    <range>
-                        <min>0.1</min>
-                        <max>200.0</max>
-                        <resolution>0.01</resolution>
-                    </range>
-                    <!-- Noise -->
-                    <noise>
-                        <type>gaussian</type>
-                        <mean>0.0</mean>
-                        <stddev>0.0025</stddev>
-                    </noise>
-                </ray>
-                <!-- Gazebo ROS plugin -->
-                <plugin name="${sensor_name}_plugin" filename="libgazebo_ros_velodyne_laser.so">
-                    <ros>
-                        <remapping>~/out:=/${sensor_name}_points</remapping>
-                    </ros>
-                    <output_type>sensor_msgs/PointCloud2</output_type>
-                    <frame_name>${sensor_name}_optical</frame_name>
-                    <organize_cloud>false</organize_cloud>
-                    <min_range>1.0</min_range>
-                    <max_range>200.0</max_range>
-                </plugin>
-            </sensor>
-        </gazebo>
-    </xacro:macro>
-</robot>
+/home/kimsohee/ev-1-5/ev-Autonomous-Vehicle-1-5/carsa_gazebo/urdf/velodyne_vlp_32c.xacro

File: install/carsa_gazebo/share/carsa_gazebo/urdf/xsens_mti3.xacro (robot description, xacro)
@@ -1,103 +1 @@
-<?xml version="1.0" ?>
-<robot xmlns:xacro="http://ros.org/wiki/xacro">
-    <!-- Xsens MTi 3 IMU -->
-    <xacro:macro name="xsens_mti3" params="parent_link sensor_name x y z roll pitch yaw">
-        <!-- Link -->
-        <link name="${sensor_name}">
-            <!-- Mesh -->
-            <visual>
-                <origin xyz="0 0 0" rpy="0 0 0" />
-                <geometry>
-                    <box size="0.035 0.035 0.01"/>
-                </geometry>
-                <material name="black">
-                    <color rgba="0.1 0.1 0.1 1.0"/>
-                </material>
-            </visual>
-        </link>
-        <!-- Joint -->
-        <joint name="${sensor_name}_joint" type="fixed">
-            <!-- Origin -->
-            <origin xyz="${x} ${y} ${z}" rpy="${radians(roll)} ${radians(pitch)} ${radians(yaw)}" />
-            <!-- Frame ID -->
-            <parent link="${parent_link}" />
-            <child link="${sensor_name}" />
-        </joint>
-        <!-- Gazebo plugin -->
-        <gazebo reference="${sensor_name}">
-            <!-- Material -->
-            <material>Gazebo/Black</material>
-            <!-- Sensor properties -->
-            <sensor name="${sensor_name}" type="imu">
-                <always_on>true</always_on>
-                <update_rate>100</update_rate>
-                <visualize>false</visualize>
-                <!-- SDFormat IMU noise model -->
-                <imu>
-                    <!-- Angular velocity (rad/s) -->
-                    <angular_velocity>
-                        <x>
-                            <noise type="gaussian">
-                                <mean>0.0</mean>
-                                <stddev>0.00005</stddev>
-                                <bias_mean>0.0</bias_mean>
-                                <bias_stddev>0.000002</bias_stddev>
-                            </noise>
-                        </x>
-                        <y>
-                            <noise type="gaussian">
-                                <mean>0.0</mean>
-                                <stddev>0.00005</stddev>
-                                <bias_mean>0.0</bias_mean>
-                                <bias_stddev>0.000002</bias_stddev>
-                            </noise>
-                        </y>
-                        <z>
-                            <noise type="gaussian">
-                                <mean>0.0</mean>
-                                <stddev>0.00005</stddev>
-                                <bias_mean>0.0</bias_mean>
-                                <bias_stddev>0.000002</bias_stddev>
-                            </noise>
-                        </z>
-                    </angular_velocity>
-                    <!-- Linear acceleration (m/s^2) -->
-                    <linear_acceleration>
-                        <x>
-                            <noise type="gaussian">
-                                <mean>0.0</mean>
-                                <stddev>0.0007</stddev>
-                                <bias_mean>0.0</bias_mean>
-                                <bias_stddev>0.0004</bias_stddev>
-                            </noise>
-                        </x>
-                        <y>
-                            <noise type="gaussian">
-                                <mean>0.0</mean>
-                                <stddev>0.0007</stddev>
-                                <bias_mean>0.0</bias_mean>
-                                <bias_stddev>0.0004</bias_stddev>
-                            </noise>
-                        </y>
-                        <z>
-                            <noise type="gaussian">
-                                <mean>0.0</mean>
-                                <stddev>0.0007</stddev>
-                                <bias_mean>0.0</bias_mean>
-                                <bias_stddev>0.0004</bias_stddev>
-                            </noise>
-                        </z>
-                    </linear_acceleration>
-                </imu>
-                <!-- Gazebo ROS plugin -->
-                <plugin name="${sensor_name}_plugin" filename="libgazebo_ros_imu_sensor.so">
-                    <ros>
-                        <remapping>~/out:=${sensor_name}/imu</remapping>
-                    </ros>
-                    <frame_name>${sensor_name}</frame_name>
-                    <initial_orientation_as_reference>false</initial_orientation_as_reference>
-                </plugin>
-            </sensor>
-        </gazebo>
-    </xacro:macro>
-</robot>
+/home/kimsohee/ev-1-5/ev-Autonomous-Vehicle-1-5/carsa_gazebo/urdf/xsens_mti3.xacro
